File: 65AcrylicKeyboard.kicad_pcb (KiCad board)
At the start: 2 copper layers, 304.8 x 123.8 mm, 153 parts, among them J1 AVR-ISP-6, J2 USB_B_Micro, K1 KEYSW, K10 KEYSW, K11 KEYSW, K12 KEYSW, K13 KEYSW, K14 KEYSW, K15 KEYSW, K16 KEYSW, K17 KEYSW, K18 KEYSW, K19 KEYSW, K2 KEYSW, K20 KEYSW, K21 KEYSW, K22 KEYSW, K23 KEYSW, K24 KEYSW, K25 KEYSW, K26 KEYSW, K27 KEYSW, K28 KEYSW, K29 KEYSW, K3 KEYSW, K30 KEYSW, K31 KEYSW, K32 KEYSW, K33 KEYSW, K34 KEYSW, K35 KEYSW, K36 KEYSW, K37 KEYSW, K38 KEYSW, K39 KEYSW, K4 KEYSW, K40 KEYSW, K41 KEYSW, K42 KEYSW, K43 KEYSW, K44 KEYSW, K45 KEYSW, K46 KEYSW, K47 KEYSW, K48 KEYSW, K49 KEYSW, K5 KEYSW, K50 KEYSW, K51 KEYSW, K52 KEYSW, K53 KEYSW, K54 KEYSW, K55 KEYSW, K56 KEYSW, K57 KEYSW, K58 KEYSW, K59 KEYSW, K6 KEYSW, K60 KEYSW, K61 KEYSW, K62 KEYSW, K63 KEYSW, K64 KEYSW, K65 KEYSW, K66 KEYSW, K67 KEYSW, K7 KEYSW, K8 KEYSW, K9 KEYSW, SW1 RESET, SW2 BOOT, U1 ATmega32A-PU-MCU_Microchip_AT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, Y1 Crystal

Commit message: Update
Parts:
- moved D6 24.8 mm to (45.2, 47.1)
- moved D7 24.8 mm to (42.1, 45.6)
- moved D16 22.7 mm to (77.8, 37.6)
- moved D11 19.1 mm to (64.3, 50.3)
- moved D19 16.2 mm to (54.8, 45.6)
- moved D15 12.8 mm to (51.6, 50.3)
- moved D12 6.55 mm to (61.1, 48.7)
- moved D14 4.49 mm to (48.4, 48.7)
- moved D13 4.49 mm to (57.9, 47.1)
Routing:
- net Net-(D15-Pad2): track 0.00 -> 100.7 mm
- net Net-(D19-Pad2): track 0.00 -> 99.6 mm
- net Net-(D14-Pad2): track 0.00 -> 79.1 mm
- net Net-(D13-Pad2): track 0.00 -> 73.2 mm
- net Net-(D7-Pad2): track 0.00 -> 56.2 mm
- net Net-(D12-Pad2): track 0.00 -> 53.4 mm
- net Net-(D11-Pad2): track 0.00 -> 32.1 mm
- net Net-(D6-Pad2): track 0.00 -> 28.5 mm
